File: 3pdt.kicad_pcb (KiCad board)
At the start: 2 copper layers, 9 parts

Commit message: Added README.
Parts:
- added G***: LOGO, Footprints:github_s, F.Cu at (132.0, 93.0)
Other:
- board text added: "Hajto/3pdt-breakeout-board"
Changed lines of the file:
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@@
 			(drillshape 0)
 			(scaleselection 1)
-			(outputdirectory "../../../Downloads/")
+			(outputdirectory "../../Downloads/")
 		)
 	)
@@
 		(embedded_fonts no)
 	)
+	(footprint "Footprints:github_s"
+		(layer "F.Cu")
+		(at 132 93)
+		(property "Reference" "G***"
+			(at 0 0 0)
+			(layer "F.SilkS")
+			(hide yes)
+			(effects
+				(font
+					(size 1.5 1.5)
+					(thickness 0.3)
+				)
+			)
+		)
+		(property "Value" "LOGO"
+			(at 0.75 0 0)
+			(layer "F.SilkS")
+			(hide yes)
+			(effects
+				(font
+					(size 1.5 1.5)
+					(thickness 0.3)
+				)
+			)
+		)
+		(property "Datasheet" ""
+			(at 0 0 0)
+			(layer "F.Fab")
+			(hide yes)
+			(effects
+				(font
+					(size 1.27 1.27)
+					(thickness 0.15)
+				)
+			)
+		)
+		(property "Description" ""
+			(at 0 0 0)
+			(layer "F.Fab")
+			(hide yes)
+			(effects
+				(font
+					(size 1.27 1.27)
+					(thickness 0.15)
+				)
+			)
+		)
+		(attr board_only exclude_from_pos_files exclude_from_bom)
+		(fp_poly
+			(pts
+				(xy -0.725766 0.859283) (xy -0.710732 0.879303) (xy -0.717351 0.894818) (xy -0.728793 0.897365)
+				(xy -0.749745 0.885118) (xy -0.752875 0.873283) (xy -0.744009 0.856627)
+			)
+			(stroke
+				(width 0)
+				(type solid)
+			)
+			(fill yes)
+			(layer "F.SilkS")
+		)
+		(fp_poly
+			(pts
+				(xy -0.92018 0.646406) (xy -0.905671 0.660074) (xy -0.904971 0.662514) (xy -0.916738 0.669046) (xy -0.92018 0.669221)
+				(xy -0.934805 0.657528) (xy -0.93539 0.653114) (xy -0.926072 0.64403)
+			)
+			(stroke
+				(width 0)
+				(type solid)
+			)
+			(fill yes)
+			(layer "F.SilkS")
+		)
+		(fp_poly
+			(pts
+				(xy -0.847034 0.707581) (xy -0.844132 0.71485) (xy -0.855049 0.729624) (xy -0.858444 0.730059) (xy -0.879043 0.719003)
+				(xy -0.882156 0.71485) (xy -0.878708 0.701829) (xy -0.867844 0.69964)
+			)
+			(stroke
+				(width 0)
+				(type solid)
+			)
+			(fill yes)
+			(layer "F.SilkS")
+		)
+		(fp_poly
+			(pts
+				(xy -0.785944 0.787863) (xy -0.783294 0.798502) (xy -0.792559 0.81945) (xy -0.813594 0.815674) (xy -0.818783 0.811177)
+				(xy -0.828471 0.788915) (xy -0.812641 0.776198) (xy -0.806108 0.775688)
+			)
+			(stroke
+				(width 0)
+				(type solid)
+			)
+			(fill yes)
+			(layer "F.SilkS")
+		)
+		(fp_poly
+			(pts
+				(xy -0.500517 0.93803) (xy -0.486253 0.952391) (xy -0.487692 0.959797) (xy -0.506052 0.971474) (xy -0.528917 0.971816)
+				(xy -0.539941 0.960738) (xy -0.528782 0.938259) (xy -0.501117 0.937804)
+			)
+			(stroke
+				(width 0)
+				(type solid)
+			)
+			(fill yes)
+			(layer "F.SilkS")
+		)
+		(fp_poly
+			(pts
+				(xy -0.381727 0.923762) (xy -0.373025 0.944756) (xy -0.390738 0.957096) (xy -0.403055 0.958203)
+				(xy -0.42778 0.952509) (xy -0.433474 0.944621) (xy -0.421339 0.927943) (xy -0.397212 0.91957)
+			)
+			(stroke
+				(width 0)
+				(type solid)
+			)
+			(fill yes)
+			(layer "F.SilkS")
+		)
+		(fp_poly
+			(pts
+				(xy -0.611698 0.925613) (xy -0.600779 0.942516) (xy -0.611788 0.956133) (xy -0.63472 0.956012) (xy -0.654435 0.942304)
+				(xy -0.654638 0.941981) (xy -0.658512 0.921262) (xy -0.656192 0.917288) (xy -0.635858 0.914308)
+			)
+			(stroke
+				(width 0)
+				(type solid)
+			)
+			(fill yes)
+			(layer "F.SilkS")
+		)
+		(fp_poly
+			(pts
+				(xy 0.206257 -1.399889) (xy 0.405348 -1.357208) (xy 0.594708 -1.288133) (xy 0.771774 -1.194354)
+				(xy 0.933983 -1.077556) (xy 1.078772 -0.939428) (xy 1.203577 -0.781656) (xy 1.305834 -0.605929)
+				(xy 1.33894 -0.533154) (xy 1.378064 -0.435204) (xy 1.40643 -0.349429) (xy 1.425608 -0.267277) (xy 1.437167 -0.180196)
+				(xy 1.442675 -0.079635) (xy 1.443725 0.038023) (xy 1.442538 0.13993) (xy 1.439515 0.218846) (xy 1.433958 0.282179)
+				(xy 1.425172 0.337337) (xy 1.41246 0.391727) (xy 1.409416 0.403053) (xy 1.340961 0.598053) (xy 1.246696 0.780537)
+				(xy 1.129003 0.947724) (xy 0.990264 1.096831) (xy 0.83286 1.225074) (xy 0.659172 1.329672) (xy 0.587558 1.363444)
+				(xy 0.515519 1.393692) (xy 0.460315 1.411829) (xy 0.419712 1.415305) (xy 0.391472 1.401572) (xy 0.373361 1.368082)
+				(xy 0.363143 1.312285) (xy 0.358581 1.231633) (xy 0.357439 1.123578) (xy 0.357425 1.101119) (xy 0.356465 0.987797)
+				(xy 0.353028 0.900085) (xy 0.346271 0.833217) (xy 0.335354 0.78243) (xy 0.319438 0.742956) (xy 0.297682 0.710032)
+				(xy 0.286044 0.696394) (xy 0.271424 0.677342) (xy 0.279245 0.670228) (xy 0.306243 0.669221) (xy 0.404672 0.657449)
+				(xy 0.510871 0.625016) (xy 0.615258 0.576245) (xy 0.70825 0.51546) (xy 0.76833 0.460726) (xy 0.831636 0.376991)
+				(xy 0.877904 0.280679) (xy 0.909776 0.165467) (xy 0.921855 0.09373) (xy 0.930496 -0.048742) (xy 0.913873 -0.177117)
+				(xy 0.871123 -0.295461) (xy 0.821287 -0.38024) (xy 0.799013 -0.417152) (xy 0.792079 -0.448621) (xy 0.797834 -0.490155)
+				(xy 0.800479 -0.501917) (xy 0.80928 -0.582506) (xy 0.804049 -0.673995) (xy 0.785872 -0.760885) (xy 0.7814 -0.774582)
+				(xy 0.768835 -0.80513) (xy 0.752724 -0.818535) (xy 0.722776 -0.819839) (xy 0.694785 -0.817012) (xy 0.650262 -0.806559)
+				(xy 0.588996 -0.785048) (xy 0.520866 -0.75614) (xy 0.487748 -0.740274) (xy 0.34982 -0.671324) (xy 0.250957 -0.692771)
+				(xy 0.190012 -0.702432) (xy 0.112079 -0.709833) (xy 0.030573 -0.713829) (xy -0.000001 -0.714217)
+				(xy -0.079183 -0.711903) (xy -0.160153 -0.705725) (xy -0.229497 -0.69683) (xy -0.250959 -0.692771)
+				(xy -0.349821 -0.671324) (xy -0.48775 -0.740274) (xy -0.555628 -0.771482) (xy -0.621515 -0.797101)
+				(xy -0.675533 -0.813467) (xy -0.694786 -0.817012) (xy -0.737576 -0.820443) (xy -0.760518 -0.814717)
+				(xy -0.773903 -0.794794) (xy -0.781401 -0.774582) (xy -0.801751 -0.690114) (xy -0.809346 -0.59831)
+				(xy -0.803102 -0.51467) (xy -0.80048 -0.501917) (xy -0.792338 -0.456186) (xy -0.796315 -0.423859)
+				(xy -0.815061 -0.38943) (xy -0.821289 -0.38024) (xy -0.884238 -0.266758) (xy -0.920413 -0.1463)
+				(xy -0.930675 -0.014801) (xy -0.921856 0.09373) (xy -0.89006 0.239967) (xy -0.838009 0.363749) (xy -0.764874 0.466028)
+				(xy -0.669826 0.547758) (xy -0.552038 0.609893) (xy -0.441685 0.645925) (xy -0.387071 0.658528)
+				(xy -0.339738 0.666987) (xy -0.316206 0.669221) (xy -0.289175 0.670636) (xy -0.281442 0.673023)
+				(xy -0.287758 0.687493) (xy -0.303975 0.720793) (xy -0.319465 0.751649) (xy -0.340662 0.79681) (xy -0.354441 0.832652)
+				(xy -0.357426 0.846174) (xy -0.372046 0.87151) (xy -0.416101 0.891462) (xy -0.479261 0.904649) (xy -0.567163 0.903905)
+				(xy -0.649249 0.877115) (xy -0.717708 0.827121) (xy -0.73006 0.813415) (xy -0.806797 0.725917) (xy -0.871665 0.662914)
+				(xy -0.927681 0.622375) (xy -0.977865 0.602269) (xy -1.025237 0.600563) (xy -1.041489 0.603879)
+				(xy -1.068084 0.619032) (xy -1.06561 0.642891) (xy -1.034108 0.675331) (xy -1.012643 0.6912) (xy -0.944003 0.754245)
+				(xy -0.884385 0.839408) (xy -0.85479 0.899446) (xy -0.808895 0.971903) (xy -0.739726 1.033324) (xy -0.69519 1.059442)
+				(xy -0.655696 1.074412) (xy -0.606171 1.083073) (xy -0.538438 1.086556) (xy -0.498114 1.086728)
+				(xy -0.357426 1.085972) (xy -0.357426 1.22633) (xy -0.360165 1.311103) (xy -0.370667 1.369201) (xy -0.392363 1.402669)
+				(xy -0.428681 1.413549) (xy -0.483051 1.403885) (xy -0.558902 1.37572) (xy -0.587559 1.363444) (xy -0.769497 1.267714)
+				(xy -0.934611 1.147594) (xy -1.081107 1.005141) (xy -1.207191 0.842412) (xy -1.311067 0.661465)
+				(xy -1.390941 0.464356) (xy -1.401771 0.430154) (xy -1.417306 0.376422) (xy -1.428374 0.32889) (xy -1.435758 0.280389)
+				(xy -1.440237 0.223749) (xy -1.442594 0.1518) (xy -1.443609 0.057374) (xy -1.443671 0.045628) (xy -1.443427 -0.059142)
+				(xy -1.441177 -0.140186) (xy -1.436409 -0.204161) (xy -1.428609 -0.257725) (xy -1.417265 -0.307535)
+				(xy -1.416124 -0.311797) (xy -1.346721 -0.513937) (xy -1.2533 -0.699754) (xy -1.137879 -0.867679)
+				(xy -1.002476 -1.016137) (xy -0.849111 -1.143558) (xy -0.679802 -1.248369) (xy -0.496568 -1.328999)
+				(xy -0.301427 -1.383876) (xy -0.096399 -1.411427) (xy -0.000001 -1.414492)
+			)
+			(stroke
+				(width 0)
+				(type solid)
+			)
+			(fill yes)
+			(layer "F.SilkS")
+		)
+		(embedded_fonts no)
+	)
 	(footprint "TestPoint:TestPoint_THTPad_1.5x1.5mm_Drill0.7mm"
 		(layer "F.Cu")
@@
 		)
 	)
+	(gr_text "Hajto/3pdt-breakeout-board"
+		(at 133.55837 93.975672 0)
+		(layer "F.SilkS")
+		(effects
+			(font
+				(size 1 1)
+				(thickness 0.1)
+			)
+			(justify left bottom)
+		)
+	)
